File: scheme/scheme/scheme.kicad_pcb (KiCad board)
At the start: 2 copper layers, 56.2 x 51 mm, 104 parts, among them IC1 ADS131M04IPWR, IC10 74HC4051D, IC2 AD8232ACPZ-R7, IC3 ESP32-S3-WROOM-1U-N16R8, IC4 AMS1117-3.3, IC5 AD8232ACPZ-R7, IC6 AD8232ACPZ-R7, IC7 AD8232ACPZ-R7, IC8 TLV9001SIDCKR, J1 Conn_01x03_Pin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

Commit message: first release 0.0.1
Parts:
- moved C5 0.26 mm to (218.0, 109.5)
- moved C7 0.26 mm to (222.7, 109.5)
- moved C8 0.26 mm to (227.2, 117.0)
- moved R22 0.26 mm to (220.2, 109.4)
- moved R24 0.26 mm to (225.1, 109.4)
- moved R28 0.26 mm to (227.1, 111.6)
- moved R29 0.26 mm to (230.4, 112.3)
- moved R30 0.26 mm to (230.4, 114.3)
- moved R31 0.26 mm to (230.5, 116.3)
- moved R32 0.26 mm to (224.3, 117.8)
- moved R33 0.26 mm to (218.6, 113.0)
- moved R34 0.26 mm to (218.6, 115.0)
- moved R35 0.26 mm to (218.6, 117.0)
- moved IC5 0.26 mm to (223.4, 114.1)
- moved R21 0.26 mm to (231.6, 109.4)
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Routing:
- net AGND: track 113.4 -> 119.8 mm
- net DGND: track 101.9 -> 105.4 mm
- net Net-(IC5-OUT): track 38.2 -> 39.0 mm
- net Net-(IC6-HPSENSE): track 22.7 -> 23.3 mm
Other:
- board text added: "1"
- board text added: "12"
- board text added: "13"
- board text added: "14"
- board text added: "16"
- board text added: "17"
- board text added: "18"
- board text added: "2"
- board text added: "21"
- board text added: "35"
- board text added: "36"
- board text added: "37"
- board text added: "38"
- board text added: "39"
- board text added: "40"
- board text added: "41"
- board text added: "42"
- board text added: "47"
- board text added: "48"
- board text added: "RX"
- board text added: "TX"
